Commit message: Add wheels and charge plate.

File: urdf/robot.urdf (robot description, URDF)
Before this commit: robot runner, 2 links, 1 joints
Links:
- added link charge_plate; visual box size=0.2 0.1 0.05
- added link left_wheel; visual cylinder length=0.1 radius=0.15
- added link right_wheel; visual cylinder length=0.1 radius=0.15
Joints:
- added joint base_to_charge: type fixed, parent base_link, child charge_plate, origin xyz=0.25 -0.225 0.07 rpy=1.5708 0 0
- added joint base_to_left_wheel: type continuous, parent base_link, child left_wheel, origin xyz=0 0.25 -0.1 rpy=-1.5708 0 0, axis 0 0 1
- added joint base_to_right_wheel: type continuous, parent base_link, child right_wheel, origin xyz=0 -0.25 -0.1 rpy=-1.5708 0 0, axis 0 0 1
- joint base_to_laser: origin xyz=0.2 0.1 0.25 rpy=0 0 0.785 -> xyz=0.3 0.1 0.25 rpy=0 0 0.785
