Commit message: Add Gazebo simulation.

File: tf2_tutorial_robot/urdf/robot.urdf (robot description, URDF)
Before this commit: robot runner, 5 links, 4 joints
Links:
- link base_link: mass None -> 15; geometry collision box size=0.6 0.6 0.35; visual box size=0.6 0.4 0.3
- link left_wheel: mass None -> 2.5
- link right_wheel: mass None -> 2.5
